File: PCB/DorMouse-V1.0.sch (EAGLE design)
At the start: 34 parts, among them IC1 LM340MP-05, IC2 MAX1551, U1 STM32F10XRXT6, X1 MINI-USB-UX60-MB-5ST

Commit message: Finished rev1.0 schematic
Parts:
- added C10: 10nF, rcl:C-EUC0402
- added C11: 1uF, rcl:C-EUC0402
- added C12, C13, C14, C15, C16, C17, C18, C19, C20, C22: 0.1uF, rcl:C-EUC0402
- BAROMETER: device Swallow:MPL115A1 -> DorMouse:MPL115A1
- C4: value 1uF -> 0.1uF
- GPS: device Swallow:UBLOX_MAX-6 -> DorMouse:UBLOX_MAX-6
- HIGH-G_ACC: device Swallow:ADXL377 -> DorMouse:ADXL377
- LOW-G_ACC: device Swallow:ADXL345 -> DorMouse:ADXL345
- XB1: device Swallow:XBEE -> DorMouse:XBEE
Connections:
- removed net MISO-3: U1PORTB_L.PB4
- removed net MOSI-3: U1PORTB_L.PB5
- removed net SCK-3: U1PORTB_L.PB3
- new net N$22: JTAG1.7
- new net N$25: JTAG1.9
- new net NRESET: JTAG1.10
- new net TCK: JTAG1.4, U1PORTA_H.PA14
- new net TDI: JTAG1.8, U1PORTA_H.PA15
- new net TDO: JTAG1.6, U1PORTB_L.PB3
- new net TMS: JTAG1.2, U1PORTA_H.PA13
- net GND: now also C10.2, C11.2, C12.1, C13.1, C14.1, C15.1, C16.1, C17.1, C18.1, C19.1, C20.1, C22.1, JTAG1.3, JTAG1.5, U1AN_POWER.VSSA
- net VCC: now also C10.1, C11.1, C12.2, C13.2, C14.2, C15.2, C16.2, C17.2, C18.2, C19.2, C20.2, C22.2, JTAG1.1, U1AN_POWER.VDDA
Other:
- moved on the sheet: C4, JMP1-0R, JMP2-0R, JTAG1, R3, R4, U1PORTA_H, U1PORTC_L
