File: PCB/DorMouse.brd (EAGLE design)
At the start: 40.9 x 69.4 mm, 56 parts, among them IC1 LM340MP-05, IC2 MAX1551, U1 STM32F10XRXT6, X1 MINI-USB-UX60-MB-5ST

Commit message: Approve errors. Add polygon Pour
Routing:
- added copper zone on layer 1, net GND
- added copper zone on layer 16, net GND
Changed lines of the file:
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@@
 <setting verticaltext="up"/>
 </settings>
-<grid distance="0.01" unitdist="mm" unit="mm" style="lines" multiple="1" display="no" altdistance="0.025" altunitdist="inch" altunit="inch"/>
+<grid distance="0.1" unitdist="mm" unit="mm" style="lines" multiple="1" display="no" altdistance="0.025" altunitdist="inch" altunit="inch"/>
 <layers>
 <layer number="1" name="Top" color="4" fill="1" visible="yes" active="yes"/>
@@
 <wire x1="25.9" y1="10.8" x2="25.57" y2="11.13" width="0.6096" layer="16"/>
 <wire x1="25.57" y1="11.13" x2="25.57" y2="23.33" width="0.6096" layer="16"/>
-<wire x1="17" y1="47.65" x2="15.95" y2="46.6" width="0" layer="19" extent="1-1"/>
+<polygon width="0.254" layer="16" isolate="0.3048" orphans="yes">
+<vertex x="0.3" y="69.2"/>
+<vertex x="0.3" y="0.3"/>
+<vertex x="40.6" y="0.3"/>
+<vertex x="40.6" y="69"/>
+<vertex x="0.5" y="69"/>
+</polygon>
+<polygon width="0.254" layer="1" isolate="0.3048" orphans="yes">
+<vertex x="0.3" y="69.1"/>
+<vertex x="0.3" y="0.2"/>
+<vertex x="40.6" y="0.2"/>
+<vertex x="40.6" y="68.9"/>
+<vertex x="0.5" y="68.9"/>
+</polygon>
 </signal>
 <signal name="VCC">
